Commit message: Retab and clean code

File: robot_description_pkg/urdf/diff_wheeled_robot_r2.xacro (robot description, xacro)
@@ -1,17 +1,17 @@
 <?xml version="1.0"?>
 <robot name="differential_wheeled_robot" xmlns:xacro="http://www.ros.org/wiki/xacro">
-	<xacro:include filename="$(find robot_description_pkg)/urdf/wheel.urdf.xacro" />
+  <xacro:include filename="$(find robot_description_pkg)/urdf/wheel.urdf.xacro" />
 <!-- Defining the colors used in this robot -->
   <material name="Black">
-	  <color rgba="0.0 0.0 0.0 1.0"/>
+    <color rgba="0.0 0.0 0.0 1.0"/>
   </material>
   <material name="Red">
-	  <color rgba="0.8 0.0 0.0 1.0"/>
+    <color rgba="0.8 0.0 0.0 1.0"/>
   </material>
   <material name="White">
-	  <color rgba="1.0 1.0 1.0 1.0"/>
+    <color rgba="1.0 1.0 1.0 1.0"/>
   </material>
   <material name="Blue">
-	  <color rgba="0.0 0.0 0.8 1.0"/>
+    <color rgba="0.0 0.0 0.8 1.0"/>
   </material>
   <!-- PROPERTY LIST -->
@@ -47,7 +47,7 @@
   <!-- Macro for calculating inertia of cylinder -->
   <macro name="cylinder_inertia" params="m r h">
-	  <inertia  ixx="${m*(3*r*r+h*h)/12}" ixy = "0" ixz = "0"
-		  iyy="${m*(3*r*r+h*h)/12}" iyz = "0"
-		  izz="${m*r*r/2}" />
+    <inertia  ixx="${m*(3*r*r+h*h)/12}" ixy = "0" ixz = "0"
+      iyy="${m*(3*r*r+h*h)/12}" iyz = "0"
+      izz="${m*r*r/2}" />
   </macro>
   <!-- the pole-->
@@ -62,247 +62,239 @@
   <!-- base_footprint is a fictitious link(frame) that is on the ground right below base_link origin -->
   <link name="base_footprint">
-	  <inertial>
-		  <mass value="0.0001" />
-		  <origin xyz="0 0 0" />
-		  <inertia ixx="0.0001" ixy="0.0" ixz="0.0"
-			  iyy="0.0001" iyz="0.0"
-			  izz="0.0001" />
-	  </inertial>
-	  <visual>
-		  <origin xyz="0 0 0" rpy="0 0 0" />
-		  <geometry>
-			  <box size="0.001 0.001 0.001" />
-		  </geometry>
-	  </visual>
+    <inertial>
+      <mass value="0.0001" />
+      <origin xyz="0 0 0" />
+      <inertia ixx="0.0001" ixy="0.0" ixz="0.0"
+        iyy="0.0001" iyz="0.0"
+        izz="0.0001" />
+    </inertial>
+    <visual>
+      <origin xyz="0 0 0" rpy="0 0 0" />
+      <geometry>
+        <box size="0.001 0.001 0.001" />
+      </geometry>
+    </visual>
   </link>
   <gazebo reference="base_footprint">
-	  <turnGravityOff>false</turnGravityOff>
+    <turnGravityOff>false</turnGravityOff>
   </gazebo>
   <joint name="base_footprint_joint" type="fixed">
-	  <origin xyz="0 1 ${wheel_radius - base_z_origin_to_wheel_origin}" rpy="0 0 0" />
-	  <parent link="base_footprint"/>
-	  <child link="base_link" />
+    <origin xyz="0 1 ${wheel_radius - base_z_origin_to_wheel_origin}" rpy="0 0 0" />
+    <parent link="base_footprint"/>
+    <child link="base_link" />
   </joint>
   <!-- BASE-LINK -->
   <!--Actual body/chassis of the robot-->
   <link name="base_link">
-	  <inertial>
-		  <mass value="${base_mass}" />
-		  <origin xyz="0 0 0" />
-		  <!--The 3x3 rotational inertia matrix. -->
-		  <cylinder_inertia  m="${base_mass}" r="${base_radius}" h="${base_height}" />
-		  <!--	<inertia ixx="1.0" ixy="0.0"  ixz="0.0"  iyy="1.0"  iyz="0.0"  izz="1.0" />
--->
-	</inertial>
-	<visual>
-		<origin xyz="0 0 0" rpy="0 0 0" />
-		<geometry>
-			<!--  <box size="${base_len} ${base_width} ${base_height}">
-				-->
-				<cylinder length="${base_height}" radius="${base_radius}" />
-			</geometry>
-			<material name="Blue" />
-		</visual>
-		<collision>
-			<origin xyz="0 0 0" rpy="0 0 0 " />
-			<geometry>
-				<!-- <box size="${base_len} ${base_width} ${base_height}">
-					-->-
-					<cylinder length="${base_height}" radius="${base_radius}" />
-				</geometry>
-			</collision>
-		</link>
-		<gazebo reference="base_link">
-			<material>Gazebo/Blue</material>
-			<turnGravityOff>false</turnGravityOff>
-		</gazebo>
-		<link name="pan_link">
-			<visual>
-				<geometry>
-					<cylinder length="${pan_link_length}" radius="${pan_link_radius}"/>
-				</geometry>
-				<origin rpy="0 0 0" xyz="0 0 0.1"/>
-				<material name="White">
-					<!--color rgba="0 0 1 1"/-->
-				</material>
-			</visual>
-			<collision>
-				<geometry>
-					<cylinder length="${pan_link_length}" radius="${pan_link_radius+0.02}"/>
-				</geometry>
-				<origin rpy="0 0 0" xyz="0 0 0.1"/>
-			</collision>
-			<xacro:inertial_matrix mass="1"/>
-		</link>
-		<gazebo reference="pan_link">
-			<material>Gazebo/White</material>
-			<turnGravityOff>false</turnGravityOff>
-		</gazebo>
-		<joint name="pan_joint" type="fixed">
-			<parent link="base_link"/>
-			<child link="pan_link"/>
-			<origin xyz="0 0 0"/>
-			<axis xyz="0 0 1" />
-			<!--limit effort="300" velocity="0.1" lower="-3.14" upper="3.14"/>
-			<dynamics damping="50" friction="1"/-->
-		</joint>
-		<gazebo reference="pan_joint">
-			<turnGravityOff>false</turnGravityOff>
-		</gazebo>
+    <inertial>
+      <mass value="${base_mass}" />
+      <origin xyz="0 0 0" />
+      <!--The 3x3 rotational inertia matrix. -->
+      <cylinder_inertia  m="${base_mass}" r="${base_radius}" h="${base_height}" />
+    </inertial>
+    <visual>
+      <origin xyz="0 0 0" rpy="0 0 0" />
+      <geometry>
+        <cylinder length="${base_height}" radius="${base_radius}" />
+      </geometry>
+      <material name="Blue" />
+    </visual>
+    <collision>
+      <origin xyz="0 0 0" rpy="0 0 0 " />
+      <geometry>
+        <cylinder length="${base_height}" radius="${base_radius}" />
+      </geometry>
+    </collision>
+  </link>
+  <gazebo reference="base_link">
+    <material>Gazebo/Blue</material>
+    <turnGravityOff>false</turnGravityOff>
+  </gazebo>
+  <link name="pan_link">
+    <visual>
+      <geometry>
+        <cylinder length="${pan_link_length}" radius="${pan_link_radius}"/>
+      </geometry>
+      <origin rpy="0 0 0" xyz="0 0 0.1"/>
+      <material name="White">
+        <!--color rgba="0 0 1 1"/-->
+      </material>
+    </visual>
+    <collision>
+      <geometry>
+        <cylinder length="${pan_link_length}" radius="${pan_link_radius+0.02}"/>
+      </geometry>
+      <origin rpy="0 0 0" xyz="0 0 0.1"/>
+    </collision>
+    <xacro:inertial_matrix mass="1"/>
+  </link>
+  <gazebo reference="pan_link">
+    <material>Gazebo/White</material>
+    <turnGravityOff>false</turnGravityOff>
+  </gazebo>
+  <joint name="pan_joint" type="fixed">
+    <parent link="base_link"/>
+    <child link="pan_link"/>
+    <origin xyz="0 0 0"/>
+    <axis xyz="0 0 1" />
+    <!--limit effort="300" velocity="0.1" lower="-3.14" upper="3.14"/>
+      <dynamics damping="50" friction="1"/-->
+    </joint>
+    <gazebo reference="pan_joint">
+      <turnGravityOff>false</turnGravityOff>
+    </gazebo>
 <!-- upper-LINK -->
   <!--Actual body/chassis of the robot-->
   <link name="upper_link">
-	  <inertial>
-		  <mass value="${base_mass}" />
-		  <origin xyz="0 0 0" />
-		  <!--The 3x3 rotational inertia matrix. -->
-		  <cylinder_inertia  m="${base_mass}" r="${base_radius2}" h="${base_height}" />
-	</inertial>
-	<visual>
-		<origin xyz="0 0 0" rpy="0 0 0" />
-		<geometry>
-				<cylinder length="${base_height}" radius="${base_radius2}" />
-			</geometry>
-			<material name="White" />
-		</visual>
-		<collision>
-			<origin xyz="0 0 0" rpy="0 0 0 " />
-			<geometry>
-				<!-- <box size="${base_len} ${base_width} ${base_height}">
-					-->-
-					<cylinder length="${base_height}" radius="${base_radius2}" />
-				</geometry>
-			</collision>
-		</link>
-		<gazebo reference="base_link">
-			<material>Gazebo/White</material>
-			<turnGravityOff>false</turnGravityOff>
-		</gazebo>
-	<joint name="upper_joint" type="fixed">
-		<parent link="pan_link"/>
-		<child link="upper_link"/>
-		<origin xyz="0 0 0.2" rpy="0 0 0"/>
-	</joint>
-	<gazebo reference="upper_joint">
-		<turnGravityOff>false</turnGravityOff>
-	</gazebo>
+    <inertial>
+      <mass value="${base_mass}" />
+      <origin xyz="0 0 0" />
+      <!--The 3x3 rotational inertia matrix. -->
+      <cylinder_inertia  m="${base_mass}" r="${base_radius2}" h="${base_height}" />
+    </inertial>
+    <visual>
+      <origin xyz="0 0 0" rpy="0 0 0" />
+      <geometry>
+        <cylinder length="${base_height}" radius="${base_radius2}" />
+      </geometry>
+      <material name="White" />
+    </visual>
+    <collision>
+      <origin xyz="0 0 0" rpy="0 0 0 " />
+      <geometry>
+        <cylinder length="${base_height}" radius="${base_radius2}" />
+      </geometry>
+    </collision>
+  </link>
+  <gazebo reference="base_link">
+    <material>Gazebo/White</material>
+    <turnGravityOff>false</turnGravityOff>
+  </gazebo>
+  <joint name="upper_joint" type="fixed">
+    <parent link="pan_link"/>
+    <child link="upper_link"/>
+    <origin xyz="0 0 0.2" rpy="0 0 0"/>
+  </joint>
+  <gazebo reference="upper_joint">
+    <turnGravityOff>false</turnGravityOff>
+  </gazebo>
 <!--frame///////////////////////////////////////////////////////
 //////////////////////////////////////////////////-->
-	<link name="frame1_link" >
-		<visual>
-			<origin xyz="0 0 0.025" rpy="0 0 0" />
-			<geometry>
-				<box size="${frame_width} ${frame_len} ${frame_height}" />
-			</geometry>
-			<material name="Blue" />
-		</visual>
-		<collision>
-			<origin xyz="0 0 0.025" rpy="0 0 0" />
-			<geometry>
-				<box size="${frame_width} ${frame_len} ${frame_height}" />
-			</geometry>
-		</collision>
-	</link>
-	<gazebo reference="frame1_link">
-		<material>Gazebo/Blue</material>
-		<turnGravityOff>false</turnGravityOff>
-	</gazebo>
-	<joint name="frame1_joint" type="fixed">
-		<parent link="upper_link"/>
-		<child link="frame1_link"/>
-		<origin xyz="0.03 0 0" rpy="0 0 0"/>
-	</joint>
-	<gazebo reference="frame1_joint">
-		<turnGravityOff>false</turnGravityOff>
-	</gazebo>
-	<link name="frame2_link" >
-		<visual>
-			<origin xyz="0 0 0.025" rpy="0 0 0" />
-			<geometry>
-				<box size="${frame_width} ${frame_len} ${frame_height}" />
-			</geometry>
-			<material name="Blue" />
-		</visual>
-		<collision>
-			<origin xyz="0 0 0.025" rpy="0 0 0" />
-			<geometry>
-				<box size="${frame_width} ${frame_len} ${frame_height}" />
-			</geometry>
-		</collision>
-	</link>
-	<gazebo reference="frame2_link">
-		<material>Gazebo/Blue</material>
-		<turnGravityOff>false</turnGravityOff>
-	</gazebo>
-	<joint name="frame2_joint" type="fixed">
-		<parent link="upper_link"/>
-		<child link="frame2_link"/>
-		<origin xyz="-0.03 0 0" rpy="0 0 0"/>
-	</joint>
-	<gazebo reference="frame1_joint">
-		<turnGravityOff>false</turnGravityOff>
-	</gazebo>
+  <link name="frame1_link" >
+    <visual>
+      <origin xyz="0 0 0.025" rpy="0 0 0" />
+      <geometry>
+        <box size="${frame_width} ${frame_len} ${frame_height}" />
+      </geometry>
+      <material name="Blue" />
+    </visual>
+    <collision>
+      <origin xyz="0 0 0.025" rpy="0 0 0" />
+      <geometry>
+        <box size="${frame_width} ${frame_len} ${frame_height}" />
+      </geometry>
+    </collision>
+  </link>
+  <gazebo reference="frame1_link">
+    <material>Gazebo/Blue</material>
+    <turnGravityOff>false</turnGravityOff>
+  </gazebo>
+  <joint name="frame1_joint" type="fixed">
+    <parent link="upper_link"/>
+    <child link="frame1_link"/>
+    <origin xyz="0.03 0 0" rpy="0 0 0"/>
+  </joint>
+  <gazebo reference="frame1_joint">
+    <turnGravityOff>false</turnGravityOff>
+  </gazebo>
+  <link name="frame2_link" >
+    <visual>
+      <origin xyz="0 0 0.025" rpy="0 0 0" />
+      <geometry>
+        <box size="${frame_width} ${frame_len} ${frame_height}" />
+      </geometry>
+      <material name="Blue" />
+    </visual>
+    <collision>
+      <origin xyz="0 0 0.025" rpy="0 0 0" />
+      <geometry>
+        <box size="${frame_width} ${frame_len} ${frame_height}" />
+      </geometry>
+    </collision>
+  </link>
+  <gazebo reference="frame2_link">
+    <material>Gazebo/Blue</material>
+    <turnGravityOff>false</turnGravityOff>
+  </gazebo>
+  <joint name="frame2_joint" type="fixed">
+    <parent link="upper_link"/>
+    <child link="frame2_link"/>
+    <origin xyz="-0.03 0 0" rpy="0 0 0"/>
+  </joint>
+  <gazebo reference="frame1_joint">
+    <turnGravityOff>false</turnGravityOff>
+  </gazebo>
 <!--Caster front  -->
-	<link name="caster_front_link">
-		<visual>
-			<origin xyz="0 0.02 0" rpy="${M_PI/2} 0 0" />
-			<geometry>
-				<sphere radius="${caster_f_radius}" />
-			</geometry>
-			<material name="Black" />
-		</visual>
-		<collision>
-			<geometry>
-				<sphere radius="${caster_f_radius}" />
-			</geometry>
-			<origin xyz="0 0.02 0" rpy="${M_PI/2} 0 0" />
-		</collision>
-		<inertial>
-			<mass value="${caster_f_mass}" />
-			<origin xyz="0 0 0" />
-			<inertia ixx="0.001" ixy="0.0" ixz="0.0"
-				iyy="0.001" iyz="0.0"
-				izz="0.001" />
-		</inertial>
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
Commit message: Z_fixed robot caster radius & odom origin in launch

File: robot_description_pkg/urdf/diff_wheeled_robot_r1.xacro (robot description, xacro)
@@ -31,10 +31,10 @@
   <!-- caster wheel mass -->
   <property name="caster_f_height" value="0.04" />
-  <property name="caster_f_radius" value="0.025" />
+  <property name="caster_f_radius" value="0.0275" />
   <property name="caster_f_mass" value="0.5" /> <!-- in kg-->
   <!-- caster wheel radius and height -->
   <!-- caster wheel mass -->
   <property name="caster_b_height" value="0.04" />
-  <property name="caster_b_radius" value="0.025" />
+  <property name="caster_b_radius" value="0.0275" />
   <property name="caster_b_mass" value="0.5" /> <!-- in kg-->
   <!-- Wheels -->
@@ -80,5 +80,5 @@
   </gazebo>
   <joint name="base_footprint_joint" type="fixed">
-    <origin xyz="0 1 ${wheel_radius - base_z_origin_to_wheel_origin}" rpy="0 0 0" />
+    <origin xyz="0 0 ${wheel_radius - base_z_origin_to_wheel_origin}" rpy="0 0 0" />
     <parent link="base_footprint"/>
     <child link="base_link" />

File: robot_description_pkg/urdf/diff_wheeled_robot_r2.xacro (robot description, xacro)
@@ -31,10 +31,10 @@
   <!-- caster wheel mass -->
   <property name="caster_f_height" value="0.04" />
-  <property name="caster_f_radius" value="0.025" />
+  <property name="caster_f_radius" value="0.0275" />
   <property name="caster_f_mass" value="0.5" /> <!-- in kg-->
   <!-- caster wheel radius and height -->
   <!-- caster wheel mass -->
   <property name="caster_b_height" value="0.04" />
-  <property name="caster_b_radius" value="0.025" />
+  <property name="caster_b_radius" value="0.0275" />
   <property name="caster_b_mass" value="0.5" /> <!-- in kg-->
   <!-- Wheels -->
@@ -80,5 +80,5 @@
   </gazebo>
   <joint name="base_footprint_joint" type="fixed">
-    <origin xyz="0 1 ${wheel_radius - base_z_origin_to_wheel_origin}" rpy="0 0 0" />
+    <origin xyz="0 0 ${wheel_radius - base_z_origin_to_wheel_origin}" rpy="0 0 0" />
     <parent link="base_footprint"/>
     <child link="base_link" />
